Commit message: WIP - fixing Ability Hand URDF

File: urdf/abilityHand/ability_hand_left_small.urdf (robot description, URDF)
Before this commit: robot ability_hand, 46 links, 45 joints
Links:
- link base: geometry collision mesh filename=package://ihmc_hands_ros2/meshes/abilityHand/palm_hull.STL; visual mesh filename=package://ihmc_hands_ros2/meshes/abilityHand/FB_palm_ref.STL
- link index_L1: geometry collision mesh filename=package://ihmc_hands_ros2/meshes/abilityHand/idx-F1-hull.STL; visual mesh filename=package://ihmc_hands_ros2/meshes/abilityHand/idx-F1.STL
- link index_L2: geometry collision mesh filename=package://ihmc_hands_ros2/meshes/abilityHand/idx-F2-hull.STL; visual mesh filename=package://ihmc_hands_ros2/meshes/abilityHand/idx-F2.STL
- link middle_L1: geometry collision mesh filename=package://ihmc_hands_ros2/meshes/abilityHand/idx-F1-hull.STL; visual mesh filename=package://ihmc_hands_ros2/meshes/abilityHand/idx-F1.STL
- link middle_L2: geometry collision mesh filename=package://ihmc_hands_ros2/meshes/abilityHand/idx-F2-hull.STL; visual mesh filename=package://ihmc_hands_ros2/meshes/abilityHand/idx-F2.STL
- link pinky_L1: geometry collision mesh filename=package://ihmc_hands_ros2/meshes/abilityHand/idx-F1-hull.STL; visual mesh filename=package://ihmc_hands_ros2/meshes/abilityHand/idx-F1.STL
- link pinky_L2: geometry collision mesh filename=package://ihmc_hands_ros2/meshes/abilityHand/idx-F2-hull.STL; visual mesh filename=package://ihmc_hands_ros2/meshes/abilityHand/idx-F2.STL
- link ring_L1: geometry collision mesh filename=package://ihmc_hands_ros2/meshes/abilityHand/idx-F1-hull.STL; visual mesh filename=package://ihmc_hands_ros2/meshes/abilityHand/idx-F1.STL
- link ring_L2: geometry collision mesh filename=package://ihmc_hands_ros2/meshes/abilityHand/idx-F2-hull.STL; visual mesh filename=package://ihmc_hands_ros2/meshes/abilityHand/idx-F2.STL
- link thumb_L1: geometry collision mesh filename=package://ihmc_hands_ros2/meshes/abilityHand/thumb-F1-hull.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; visual mesh filename=package://ihmc_hands_ros2/meshes/abilityHand/thumb-F1.STL
- link thumb_L2: geometry collision mesh filename=package://ihmc_hands_ros2/meshes/abilityHand/thumb-F2-hull.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; visual mesh filename=package://ihmc_hands_ros2/meshes/abilityHand/thumb-F2-left.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

File: urdf/abilityHand/ability_hand_right_large.urdf (robot description, URDF)
Before this commit: robot ability_hand, 46 links, 45 joints
Links:
- link base: geometry collision mesh filename=package://ihmc_hands_ros2/meshes/abilityHand/palm_hull_mir.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; visual mesh filename=package://ihmc_hands_ros2/meshes/abilityHand/FB_palm_ref_MI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
- link index_L1: geometry collision mesh filename=package://ihmc_hands_ros2/meshes/abilityHand/idx-F1-hull.STL; visual mesh filename=package://ihmc_hands_ros2/meshes/abilityHand/idx-F1.STL
- link index_L2: geometry collision mesh filename=package://ihmc_hands_ros2/meshes/abilityHand/idx-F2-Lg-hull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; visual mesh filename=package://ihmc_hands_ros2/meshes/abilityHand/idx-F2-Lg.STL
- link middle_L1: geometry collision mesh filename=package://ihmc_hands_ros2/meshes/abilityHand/idx-F1-hull.STL; visual mesh filename=package://ihmc_hands_ros2/meshes/abilityHand/idx-F1.STL
- link middle_L2: geometry collision mesh filename=package://ihmc_hands_ros2/meshes/abilityHand/idx-F2-Lg-hull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; visual mesh filename=package://ihmc_hands_ros2/meshes/abilityHand/idx-F2-Lg.STL
- link pinky_L1: geometry collision mesh filename=package://ihmc_hands_ros2/meshes/abilityHand/idx-F1-hull.STL; visual mesh filename=package://ihmc_hands_ros2/meshes/abilityHand/idx-F1.STL
- link pinky_L2: geometry collision mesh filename=package://ihmc_hands_ros2/meshes/abilityHand/idx-F2-hull.STL; visual mesh filename=package://ihmc_hands_ros2/meshes/abilityHand/idx-F2.STL
- link ring_L1: geometry collision mesh filename=package://ihmc_hands_ros2/meshes/abilityHand/idx-F1-hull.STL; visual mesh filename=package://ihmc_hands_ros2/meshes/abilityHand/idx-F1.STL
- link ring_L2: geometry collision mesh filename=package://ihmc_hands_ros2/meshes/abilityHand/idx-F2-Lg-hull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; visual mesh filename=package://ihmc_hands_ros2/meshes/abilityHand/idx-F2-Lg.STL
- link thumb_L1: geometry collision mesh filename=package://ihmc_hands_ros2/meshes/abilityHand/thumb-F1-MIR-h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; visual mesh filename=package://ihmc_hands_ros2/meshes/abilityHand/thumb-F1-MIR.S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
- link thumb_L2: geometry collision mesh filename=package://ihmc_hands_ros2/meshes/abilityHand/thumb-F2-hull.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; visual mesh filename=package://ihmc_hands_ros2/meshes/abilityHand/thumb-F2-right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

File: urdf/abilityHand/ability_hand_right_large_no_fsr.urdf (robot description, URDF)
Before this commit: robot ability_hand, 16 links, 15 joints
Links:
- link base: geometry collision mesh filename=package://ihmc_hands_ros2/meshes/abilityHand/palm_hull_mir.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; visual mesh filename=package://ihmc_hands_ros2/meshes/abilityHand/FB_palm_ref_MI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
- link index_L1: geometry collision mesh filename=package://ihmc_hands_ros2/meshes/abilityHand/idx-F1-hull.STL; visual mesh filename=package://ihmc_hands_ros2/meshes/abilityHand/idx-F1.STL
- link index_L2: geometry collision mesh filename=package://ihmc_hands_ros2/meshes/abilityHand/idx-F2-Lg-hull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; visual mesh filename=package://ihmc_hands_ros2/meshes/abilityHand/idx-F2-Lg.STL
- link middle_L1: geometry collision mesh filename=package://ihmc_hands_ros2/meshes/abilityHand/idx-F1-hull.STL; visual mesh filename=package://ihmc_hands_ros2/meshes/abilityHand/idx-F1.STL
- link middle_L2: geometry collision mesh filename=package://ihmc_hands_ros2/meshes/abilityHand/idx-F2-Lg-hull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; visual mesh filename=package://ihmc_hands_ros2/meshes/abilityHand/idx-F2-Lg.STL
- link pinky_L1: geometry collision mesh filename=package://ihmc_hands_ros2/meshes/abilityHand/idx-F1-hull.STL; visual mesh filename=package://ihmc_hands_ros2/meshes/abilityHand/idx-F1.STL
- link pinky_L2: geometry collision mesh filename=package://ihmc_hands_ros2/meshes/abilityHand/idx-F2-hull.STL; visual mesh filename=package://ihmc_hands_ros2/meshes/abilityHand/idx-F2.STL
- link ring_L1: geometry collision mesh filename=package://ihmc_hands_ros2/meshes/abilityHand/idx-F1-hull.STL; visual mesh filename=package://ihmc_hands_ros2/meshes/abilityHand/idx-F1.STL
- link ring_L2: geometry collision mesh filename=package://ihmc_hands_ros2/meshes/abilityHand/idx-F2-Lg-hull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; visual mesh filename=package://ihmc_hands_ros2/meshes/abilityHand/idx-F2-Lg.STL
- link thumb_L1: geometry collision mesh filename=package://ihmc_hands_ros2/meshes/abilityHand/thumb-F1-MIR-h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; visual mesh filename=package://ihmc_hands_ros2/meshes/abilityHand/thumb-F1-MIR.S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
- link thumb_L2: geometry collision mesh filename=package://ihmc_hands_ros2/meshes/abilityHand/thumb-F2-hull.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; visual mesh filename=package://ihmc_hands_ros2/meshes/abilityHand/thumb-F2-right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

File: urdf/abilityHand/ability_hand_right_small.urdf (robot description, URDF)
Before this commit: robot ability_hand, 46 links, 45 joints
Links:
- link base: geometry collision mesh filename=package://ihmc_hands_ros2/meshes/abilityHand/palm_hull_mir.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; visual mesh filename=package://ihmc_hands_ros2/meshes/abilityHand/FB_palm_ref_MI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
- link index_L1: geometry collision mesh filename=package://ihmc_hands_ros2/meshes/abilityHand/idx-F1-hull.STL; visual mesh filename=package://ihmc_hands_ros2/meshes/abilityHand/idx-F1.STL
- link index_L2: geometry collision mesh filename=package://ihmc_hands_ros2/meshes/abilityHand/idx-F2-hull.STL; visual mesh filename=package://ihmc_hands_ros2/meshes/abilityHand/idx-F2.STL
- link middle_L1: geometry collision mesh filename=package://ihmc_hands_ros2/meshes/abilityHand/idx-F1-hull.STL; visual mesh filename=package://ihmc_hands_ros2/meshes/abilityHand/idx-F1.STL
- link middle_L2: geometry collision mesh filename=package://ihmc_hands_ros2/meshes/abilityHand/idx-F2-hull.STL; visual mesh filename=package://ihmc_hands_ros2/meshes/abilityHand/idx-F2.STL
- link pinky_L1: geometry collision mesh filename=package://ihmc_hands_ros2/meshes/abilityHand/idx-F1-hull.STL; visual mesh filename=package://ihmc_hands_ros2/meshes/abilityHand/idx-F1.STL
- link pinky_L2: geometry collision mesh filename=package://ihmc_hands_ros2/meshes/abilityHand/idx-F2-hull.STL; visual mesh filename=package://ihmc_hands_ros2/meshes/abilityHand/idx-F2.STL
- link ring_L1: geometry collision mesh filename=package://ihmc_hands_ros2/meshes/abilityHand/idx-F1-hull.STL; visual mesh filename=package://ihmc_hands_ros2/meshes/abilityHand/idx-F1.STL
- link ring_L2: geometry collision mesh filename=package://ihmc_hands_ros2/meshes/abilityHand/idx-F2-hull.STL; visual mesh filename=package://ihmc_hands_ros2/meshes/abilityHand/idx-F2.STL
- link thumb_L1: geometry collision mesh filename=package://ihmc_hands_ros2/meshes/abilityHand/thumb-F1-MIR-h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; visual mesh filename=package://ihmc_hands_ros2/meshes/abilityHand/thumb-F1-MIR.S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
- link thumb_L2: geometry collision mesh filename=package://ihmc_hands_ros2/meshes/abilityHand/thumb-F2-hull.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; visual mesh filename=package://ihmc_hands_ros2/meshes/abilityHand/thumb-F2-right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
