Commit message: Fix right large pinky mesh url.

File: urdf/abilityHand/ability_hand_right_large.urdf (robot description, URDF)
Before this commit: robot right_ability_hand, 46 links, 45 joints
Links:
- link right_ability_hand_pinky_L2: geometry collision mesh filename=package://abilityHand/idx-F2-hull.obj; visual mesh filename=package://abilityHand/idx-F2-Lg.obj
