Commit message: Reorganize URDFs and meshes

File: urdf/ezGripper/left_ezgripper_gen2.urdf (robot description, URDF)
Before this commit: robot right_ezgripper_gen2, 5 links, 4 joints
Links:
- removed link right_ezgripper_finger_l1_1
- removed link right_ezgripper_finger_l1_2
- removed link right_ezgripper_finger_l2_1
- removed link right_ezgripper_finger_l2_2
- removed link right_ezgripper_palm_link
- added link left_ezgripper_finger_l1_1, mass 0.025; collision mesh filename=package://ezGripper/ezgripper_gen2/SAKE_Finger_L1_Gen2.obj; visual mesh filename=package://ezGripper/ezgripper_gen2/SAKE_Finger_L1_Gen2.obj
- added link left_ezgripper_finger_l1_2, mass 0.025; collision mesh filename=package://ezGripper/ezgripper_gen2/SAKE_Finger_L1_Gen2.obj; visual mesh filename=package://ezGripper/ezgripper_gen2/SAKE_Finger_L1_Gen2.obj
- added link left_ezgripper_finger_l2_1, mass .025; collision mesh filename=package://ezGripper/ezgripper_gen2/SAKE_Finger_L2_Gen2.obj; visual mesh filename=package://ezGripper/ezgripper_gen2/SAKE_Finger_L2_Gen2.obj
- added link left_ezgripper_finger_l2_2, mass .025; collision mesh filename=package://ezGripper/ezgripper_gen2/SAKE_Finger_L2_Gen2.obj; visual mesh filename=package://ezGripper/ezgripper_gen2/SAKE_Finger_L2_Gen2.obj
- added link left_ezgripper_palm_link, mass 0.3; collision mesh filename=package://ezGripper/ezgripper_gen2/SAKE_Palm_Dual_Gen2.obj; visual mesh filename=package://ezGripper/ezgripper_gen2/SAKE_Palm_Dual_Gen2.obj
Joints:
- removed joint right_ezgripper_knuckle_l1_l2_1
- removed joint right_ezgripper_knuckle_l1_l2_2
- removed joint right_ezgripper_knuckle_palm_l1_1
- removed joint right_ezgripper_knuckle_palm_l1_2
- added joint left_ezgripper_knuckle_l1_l2_1: type revolute, parent left_ezgripper_finger_l1_1, child left_ezgripper_finger_l2_1, origin xyz=0.052 0 0 rpy=0 0 0, axis 0 1 0, limit lower=0 upper=1.94 effort=1 velocity=3.67
- added joint left_ezgripper_knuckle_l1_l2_2: type revolute, parent left_ezgripper_finger_l1_2, child left_ezgripper_finger_l2_2, origin xyz=0.052 0 0 rpy=0 0 0, axis 0 1 0, limit lower=0 upper=1.94 effort=1 velocity=3.67, mimic joint=left_ezgripper_knuckle_l1_l2_1
- added joint left_ezgripper_knuckle_palm_l1_1: type revolute, parent left_ezgripper_palm_link, child left_ezgripper_finger_l1_1, origin xyz=0.072569 0.03 0 rpy=-1.5708 0 1.57075, axis 0 1 0, limit lower=0 upper=1.94 effort=1 velocity=3.67
- added joint left_ezgripper_knuckle_palm_l1_2: type revolute, parent left_ezgripper_palm_link, child left_ezgripper_finger_l1_2, origin xyz=0.072569 -0.03 0 rpy=1.5708 0 -1.57075, axis 0 1 0, limit lower=0 upper=1.94 effort=1 velocity=3.67, mimic joint=left_ezgripper_knuckle_palm_l1_1

File: urdf/ezGripper/right_ezgripper_gen2.urdf (robot description, URDF)
Before this commit: robot left_ezgripper_gen2, 5 links, 4 joints
Links:
- removed link left_ezgripper_finger_l1_1
- removed link left_ezgripper_finger_l1_2
- removed link left_ezgripper_finger_l2_1
- removed link left_ezgripper_finger_l2_2
- removed link left_ezgripper_palm_link
- added link right_ezgripper_finger_l1_1, mass 0.025; collision mesh filename=package://ezGripper/ezgripper_gen2/SAKE_Finger_L1_Gen2.obj; visual mesh filename=package://ezGripper/ezgripper_gen2/SAKE_Finger_L1_Gen2.obj
- added link right_ezgripper_finger_l1_2, mass 0.025; collision mesh filename=package://ezGripper/ezgripper_gen2/SAKE_Finger_L1_Gen2.obj; visual mesh filename=package://ezGripper/ezgripper_gen2/SAKE_Finger_L1_Gen2.obj
- added link right_ezgripper_finger_l2_1, mass .025; collision mesh filename=package://ezGripper/ezgripper_gen2/SAKE_Finger_L2_Gen2.obj; visual mesh filename=package://ezGripper/ezgripper_gen2/SAKE_Finger_L2_Gen2.obj
- added link right_ezgripper_finger_l2_2, mass .025; collision mesh filename=package://ezGripper/ezgripper_gen2/SAKE_Finger_L2_Gen2.obj; visual mesh filename=package://ezGripper/ezgripper_gen2/SAKE_Finger_L2_Gen2.obj
- added link right_ezgripper_palm_link, mass 0.3; collision mesh filename=package://ezGripper/ezgripper_gen2/SAKE_Palm_Dual_Gen2.obj; visual mesh filename=package://ezGripper/ezgripper_gen2/SAKE_Palm_Dual_Gen2.obj
Joints:
- removed joint left_ezgripper_knuckle_l1_l2_1
- removed joint left_ezgripper_knuckle_l1_l2_2
- removed joint left_ezgripper_knuckle_palm_l1_1
- removed joint left_ezgripper_knuckle_palm_l1_2
- added joint right_ezgripper_knuckle_l1_l2_1: type revolute, parent right_ezgripper_finger_l1_1, child right_ezgripper_finger_l2_1, origin xyz=0.052 0 0 rpy=0 0 0, axis 0 1 0, limit lower=0 upper=1.94 effort=1 velocity=3.67
- added joint right_ezgripper_knuckle_l1_l2_2: type revolute, parent right_ezgripper_finger_l1_2, child right_ezgripper_finger_l2_2, origin xyz=0.052 0 0 rpy=0 0 0, axis 0 1 0, limit lower=0 upper=1.94 effort=1 velocity=3.67, mimic joint=right_ezgripper_knuckle_l1_l2_1
- added joint right_ezgripper_knuckle_palm_l1_1: type revolute, parent right_ezgripper_palm_link, child right_ezgripper_finger_l1_1, origin xyz=0.072569 0.03 0 rpy=-1.5708 0 1.57075, axis 0 1 0, limit lower=0 upper=1.94 effort=1 velocity=3.67
- added joint right_ezgripper_knuckle_palm_l1_2: type revolute, parent right_ezgripper_palm_link, child right_ezgripper_finger_l1_2, origin xyz=0.072569 -0.03 0 rpy=1.5708 0 -1.57075, axis 0 1 0, limit lower=0 upper=1.94 effort=1 velocity=3.67, mimic joint=right_ezgripper_knuckle_palm_l1_1

Commit message: Fixed Ability Hand mimic joints

File: urdf/abilityHand/ability_hand_left_large.urdf (robot description, URDF)
Before this commit: robot left_ability_hand, 46 links, 45 joints
Joints:
- joint left_ability_hand_index_q2: mimic joint=index_q1 multiplier=1.05851325 offset=0.72349796 -> joint=left_ability_hand_index_q1 multiplier=1.05851325 offset=0.72349796
- joint left_ability_hand_middle_q2: mimic joint=middle_q1 multiplier=1.05851325 offset=0.72349796 -> joint=left_ability_hand_middle_q1 multiplier=1.05851325 offset=0.72349796
- joint left_ability_hand_pinky_q2: mimic joint=pinky_q1 multiplier=1.05851325 offset=0.72349796 -> joint=left_ability_hand_pinky_q1 multiplier=1.05851325 offset=0.72349796
- joint left_ability_hand_ring_q2: mimic joint=ring_q1 multiplier=1.05851325 offset=0.72349796 -> joint=left_ability_hand_ring_q1 multiplier=1.05851325 offset=0.72349796

File: urdf/abilityHand/ability_hand_left_small.urdf (robot description, URDF)
Before this commit: robot left_ability_hand, 46 links, 45 joints
Joints:
- joint left_ability_hand_index_q2: mimic joint=index_q1 multiplier=1.05851325 offset=0.72349796 -> joint=left_ability_hand_index_q1 multiplier=1.05851325 offset=0.72349796
- joint left_ability_hand_middle_q2: mimic joint=middle_q1 multiplier=1.05851325 offset=0.72349796 -> joint=left_ability_hand_middle_q1 multiplier=1.05851325 offset=0.72349796
- joint left_ability_hand_pinky_q2: mimic joint=pinky_q1 multiplier=1.05851325 offset=0.72349796 -> joint=left_ability_hand_pinky_q1 multiplier=1.05851325 offset=0.72349796
- joint left_ability_hand_ring_q2: mimic joint=ring_q1 multiplier=1.05851325 offset=0.72349796 -> joint=left_ability_hand_ring_q1 multiplier=1.05851325 offset=0.72349796

File: urdf/abilityHand/ability_hand_right_large.urdf (robot description, URDF)
Before this commit: robot right_ability_hand, 46 links, 45 joints
Joints:
- joint right_ability_hand_index_q2: mimic joint=index_q1 multiplier=1.05851325 offset=0.72349796 -> joint=right_ability_hand_index_q1 multiplier=1.05851325 offset=0.72349796
- joint right_ability_hand_middle_q2: mimic joint=middle_q1 multiplier=1.05851325 offset=0.72349796 -> joint=right_ability_hand_middle_q1 multiplier=1.05851325 offset=0.72349796
- joint right_ability_hand_pinky_q2: mimic joint=pinky_q1 multiplier=1.05851325 offset=0.72349796 -> joint=right_ability_hand_pinky_q1 multiplier=1.05851325 offset=0.72349796
- joint right_ability_hand_ring_q2: mimic joint=ring_q1 multiplier=1.05851325 offset=0.72349796 -> joint=right_ability_hand_ring_q1 multiplier=1.05851325 offset=0.72349796

File: urdf/abilityHand/ability_hand_right_large_no_fsr.urdf (robot description, URDF)
Before this commit: robot right_ability_hand, 16 links, 15 joints
Joints:
- joint right_ability_hand_index_q2: mimic joint=index_q1 multiplier=1.05851325 offset=0.72349796 -> joint=right_ability_hand_index_q1 multiplier=1.05851325 offset=0.72349796
- joint right_ability_hand_middle_q2: mimic joint=middle_q1 multiplier=1.05851325 offset=0.72349796 -> joint=right_ability_hand_middle_q1 multiplier=1.05851325 offset=0.72349796
- joint right_ability_hand_pinky_q2: mimic joint=pinky_q1 multiplier=1.05851325 offset=0.72349796 -> joint=right_ability_hand_pinky_q1 multiplier=1.05851325 offset=0.72349796
- joint right_ability_hand_ring_q2: mimic joint=ring_q1 multiplier=1.05851325 offset=0.72349796 -> joint=right_ability_hand_ring_q1 multiplier=1.05851325 offset=0.72349796

File: urdf/abilityHand/ability_hand_right_small.urdf (robot description, URDF)
Before this commit: robot right_ability_hand, 46 links, 45 joints
Joints:
- joint right_ability_hand_index_q2: mimic joint=index_q1 multiplier=1.05851325 offset=0.72349796 -> joint=right_ability_hand_index_q1 multiplier=1.05851325 offset=0.72349796
- joint right_ability_hand_middle_q2: mimic joint=middle_q1 multiplier=1.05851325 offset=0.72349796 -> joint=right_ability_hand_middle_q1 multiplier=1.05851325 offset=0.72349796
- joint right_ability_hand_pinky_q2: mimic joint=pinky_q1 multiplier=1.05851325 offset=0.72349796 -> joint=right_ability_hand_pinky_q1 multiplier=1.05851325 offset=0.72349796
- joint right_ability_hand_ring_q2: mimic joint=ring_q1 multiplier=1.05851325 offset=0.72349796 -> joint=right_ability_hand_ring_q1 multiplier=1.05851325 offset=0.72349796

Commit message: Use lower poly meshes in URDF

File: urdf/abilityHand/ability_hand_left_large.urdf (robot description, URDF)
Before this commit: robot left_ability_hand, 46 links, 45 joints
Links:
- link left_ability_hand_base: geometry collision mesh filename=package://abilityHand/palm_hull.obj; visual mesh filename=package://abilityHand/FB_palm_ref_lp.obj

File: urdf/abilityHand/ability_hand_left_small.urdf (robot description, URDF)
Before this commit: robot left_ability_hand, 46 links, 45 joints
Links:
- link left_ability_hand_base: geometry collision mesh filename=package://abilityHand/palm_hull.obj; visual mesh filename=package://abilityHand/FB_palm_ref_lp.obj

File: urdf/abilityHand/ability_hand_right_large.urdf (robot description, URDF)
Before this commit: robot right_ability_hand, 46 links, 45 joints
Links:
- link right_ability_hand_base: geometry collision mesh filename=package://abilityHand/palm_hull_mir.obj; visual mesh filename=package://abilityHand/FB_palm_ref_MIR_lp.obj

File: urdf/abilityHand/ability_hand_right_large_no_fsr.urdf (robot description, URDF)
Before this commit: robot right_ability_hand, 16 links, 15 joints
Links:
- link right_ability_hand_base: geometry collision mesh filename=package://abilityHand/palm_hull_mir.obj; visual mesh filename=package://abilityHand/FB_palm_ref_MIR_lp.obj

File: urdf/abilityHand/ability_hand_right_small.urdf (robot description, URDF)
Before this commit: robot right_ability_hand, 46 links, 45 joints
Links:
- link right_ability_hand_base: geometry collision mesh filename=package://abilityHand/palm_hull_mir.obj; visual mesh filename=package://abilityHand/FB_palm_ref_MIR_lp.obj
