Commit message: Fix hand models

File: urdf/ezGripper/left_ezgripper_gen2.urdf (robot description, URDF)
Before this commit: robot left_ezgripper_gen2, 5 links, 4 joints
Links:
- removed link left_ezgripper_finger_L1_1
- removed link left_ezgripper_finger_L1_2
- removed link left_ezgripper_finger_L2_1
- removed link left_ezgripper_finger_L2_2
- added link left_ezgripper_finger_l1_1, mass 0.025; collision mesh filename=package://ihmc_hands_ros2/meshes/ezGripper/ezgripper_gen2/S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; visual mesh filename=package://ihmc_hands_ros2/meshes/ezGripper/ezgripper_gen2/S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
- added link left_ezgripper_finger_l1_2, mass 0.025; collision mesh filename=package://ihmc_hands_ros2/meshes/ezGripper/ezgripper_gen2/S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; visual mesh filename=package://ihmc_hands_ros2/meshes/ezGripper/ezgripper_gen2/S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
- added link left_ezgripper_finger_l2_1, mass .025; collision mesh filename=package://ihmc_hands_ros2/meshes/ezGripper/ezgripper_gen2/S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; visual mesh filename=package://ihmc_hands_ros2/meshes/ezGripper/ezgripper_gen2/S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
- added link left_ezgripper_finger_l2_2, mass .025; collision mesh filename=package://ihmc_hands_ros2/meshes/ezGripper/ezgripper_gen2/S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; visual mesh filename=package://ihmc_hands_ros2/meshes/ezGripper/ezgripper_gen2/S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
Joints:
- removed joint left_ezgripper_knuckle_L1_L2_1
- removed joint left_ezgripper_knuckle_L1_L2_2
- removed joint left_ezgripper_knuckle_palm_L1_1
- removed joint left_ezgripper_knuckle_palm_L1_2
- added joint left_ezgripper_knuckle_l1_l2_1: type revolute, parent left_ezgripper_finger_l1_1, child left_ezgripper_finger_l2_1, origin xyz=0.052 0 0 rpy=0 0 0, axis 0 1 0, limit lower=0 upper=1.94 effort=1 velocity=3.67
- added joint left_ezgripper_knuckle_l1_l2_2: type revolute, parent left_ezgripper_finger_l1_2, child left_ezgripper_finger_l2_2, origin xyz=0.052 0 0 rpy=0 0 0, axis 0 1 0, limit lower=0 upper=1.94 effort=1 velocity=3.67, mimic joint=left_ezgripper_knuckle_l1_l2_1
- added joint left_ezgripper_knuckle_palm_l1_1: type revolute, parent left_ezgripper_palm_link, child left_ezgripper_finger_l1_1, origin xyz=0.072569 0.03 0 rpy=-1.5708 0 1.57075, axis 0 1 0, limit lower=0 upper=1.94 effort=1 velocity=3.67
- added joint left_ezgripper_knuckle_palm_l1_2: type revolute, parent left_ezgripper_palm_link, child left_ezgripper_finger_l1_2, origin xyz=0.072569 -0.03 0 rpy=1.5708 0 -1.57075, axis 0 1 0, limit lower=0 upper=1.94 effort=1 velocity=3.67, mimic joint=left_ezgripper_knuckle_palm_l1_1

File: urdf/ezGripper/right_ezgripper_gen2.urdf (robot description, URDF)
Before this commit: robot right_ezgripper_gen2, 5 links, 4 joints
Links:
- removed link right_ezgripper_finger_L1_1
- removed link right_ezgripper_finger_L1_2
- removed link right_ezgripper_finger_L2_1
- removed link right_ezgripper_finger_L2_2
- added link right_ezgripper_finger_l1_1, mass 0.025; collision mesh filename=package://ihmc_hands_ros2/meshes/ezGripper/ezgripper_gen2/S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; visual mesh filename=package://ihmc_hands_ros2/meshes/ezGripper/ezgripper_gen2/S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
- added link right_ezgripper_finger_l1_2, mass 0.025; collision mesh filename=package://ihmc_hands_ros2/meshes/ezGripper/ezgripper_gen2/S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; visual mesh filename=package://ihmc_hands_ros2/meshes/ezGripper/ezgripper_gen2/S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
- added link right_ezgripper_finger_l2_1, mass .025; collision mesh filename=package://ihmc_hands_ros2/meshes/ezGripper/ezgripper_gen2/S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; visual mesh filename=package://ihmc_hands_ros2/meshes/ezGripper/ezgripper_gen2/S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
- added link right_ezgripper_finger_l2_2, mass .025; collision mesh filename=package://ihmc_hands_ros2/meshes/ezGripper/ezgripper_gen2/S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; visual mesh filename=package://ihmc_hands_ros2/meshes/ezGripper/ezgripper_gen2/S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
Joints:
- removed joint right_ezgripper_knuckle_L1_L2_1
- removed joint right_ezgripper_knuckle_L1_L2_2
- removed joint right_ezgripper_knuckle_palm_L1_1
- removed joint right_ezgripper_knuckle_palm_L1_2
- added joint right_ezgripper_knuckle_l1_l2_1: type revolute, parent right_ezgripper_finger_l1_1, child right_ezgripper_finger_l2_1, origin xyz=0.052 0 0 rpy=0 0 0, axis 0 1 0, limit lower=0 upper=1.94 effort=1 velocity=3.67
- added joint right_ezgripper_knuckle_l1_l2_2: type revolute, parent right_ezgripper_finger_l1_2, child right_ezgripper_finger_l2_2, origin xyz=0.052 0 0 rpy=0 0 0, axis 0 1 0, limit lower=0 upper=1.94 effort=1 velocity=3.67, mimic joint=right_ezgripper_knuckle_l1_l2_1
- added joint right_ezgripper_knuckle_palm_l1_1: type revolute, parent right_ezgripper_palm_link, child right_ezgripper_finger_l1_1, origin xyz=0.072569 0.03 0 rpy=-1.5708 0 1.57075, axis 0 1 0, limit lower=0 upper=1.94 effort=1 velocity=3.67
- added joint right_ezgripper_knuckle_palm_l1_2: type revolute, parent right_ezgripper_palm_link, child right_ezgripper_finger_l1_2, origin xyz=0.072569 -0.03 0 rpy=1.5708 0 -1.57075, axis 0 1 0, limit lower=0 upper=1.94 effort=1 velocity=3.67, mimic joint=right_ezgripper_knuckle_palm_l1_1
