Commit message: modified hand urdf/mesh paths to be consistant with our typical system

File: hand-models/abilityHand/urdf/ability_hand_left_large.urdf (robot description, URDF)
Before this commit: robot left_ability_hand, 46 links, 45 joints
Links:
- link left_ability_hand_base: geometry collision mesh filename=package://abilityHand/meshes/palm_hull.STL; visual mesh filename=package://abilityHand/meshes/FB_palm_ref.STL
- link left_ability_hand_index_L1: geometry collision mesh filename=package://abilityHand/meshes/idx-F1-hull.STL; visual mesh filename=package://abilityHand/meshes/idx-F1.STL
- link left_ability_hand_index_L2: geometry collision mesh filename=package://abilityHand/meshes/idx-F2-Lg-hull.STL; visual mesh filename=package://abilityHand/meshes/idx-F2-Lg.STL
- link left_ability_hand_middle_L1: geometry collision mesh filename=package://abilityHand/meshes/idx-F1-hull.STL; visual mesh filename=package://abilityHand/meshes/idx-F1.STL
- link left_ability_hand_middle_L2: geometry collision mesh filename=package://abilityHand/meshes/idx-F2-Lg-hull.STL; visual mesh filename=package://abilityHand/meshes/idx-F2-Lg.STL
- link left_ability_hand_pinky_L1: geometry collision mesh filename=package://abilityHand/meshes/idx-F1-hull.STL; visual mesh filename=package://abilityHand/meshes/idx-F1.STL
- link left_ability_hand_pinky_L2: geometry collision mesh filename=package://abilityHand/meshes/idx-F2-hull.STL; visual mesh filename=package://abilityHand/meshes/idx-F2-Lg.STL
- link left_ability_hand_ring_L1: geometry collision mesh filename=package://abilityHand/meshes/idx-F1-hull.STL; visual mesh filename=package://abilityHand/meshes/idx-F1.STL
- link left_ability_hand_ring_L2: geometry collision mesh filename=package://abilityHand/meshes/idx-F2-Lg-hull.STL; visual mesh filename=package://abilityHand/meshes/idx-F2-Lg.STL
- link left_ability_hand_thumb_L1: geometry collision mesh filename=package://abilityHand/meshes/thumb-F1-hull.STL; visual mesh filename=package://abilityHand/meshes/thumb-F1.STL
- link left_ability_hand_thumb_L2: geometry collision mesh filename=package://abilityHand/meshes/thumb-F2-hull.STL; visual mesh filename=package://abilityHand/meshes/thumb-F2-left.STL

File: hand-models/abilityHand/urdf/ability_hand_left_small.urdf (robot description, URDF)
Before this commit: robot left_ability_hand, 46 links, 45 joints
Links:
- link left_ability_hand_base: geometry collision mesh filename=package://abilityHand/meshes/palm_hull.STL; visual mesh filename=package://abilityHand/meshes/FB_palm_ref.STL
- link left_ability_hand_index_L1: geometry collision mesh filename=package://abilityHand/meshes/idx-F1-hull.STL; visual mesh filename=package://abilityHand/meshes/idx-F1.STL
- link left_ability_hand_index_L2: geometry collision mesh filename=package://abilityHand/meshes/idx-F2-hull.STL; visual mesh filename=package://abilityHand/meshes/idx-F2.STL
- link left_ability_hand_middle_L1: geometry collision mesh filename=package://abilityHand/meshes/idx-F1-hull.STL; visual mesh filename=package://abilityHand/meshes/idx-F1.STL
- link left_ability_hand_middle_L2: geometry collision mesh filename=package://abilityHand/meshes/idx-F2-hull.STL; visual mesh filename=package://abilityHand/meshes/idx-F2.STL
- link left_ability_hand_pinky_L1: geometry collision mesh filename=package://abilityHand/meshes/idx-F1-hull.STL; visual mesh filename=package://abilityHand/meshes/idx-F1.STL
- link left_ability_hand_pinky_L2: geometry collision mesh filename=package://abilityHand/meshes/idx-F2-hull.STL; visual mesh filename=package://abilityHand/meshes/idx-F2.STL
- link left_ability_hand_ring_L1: geometry collision mesh filename=package://abilityHand/meshes/idx-F1-hull.STL; visual mesh filename=package://abilityHand/meshes/idx-F1.STL
- link left_ability_hand_ring_L2: geometry collision mesh filename=package://abilityHand/meshes/idx-F2-hull.STL; visual mesh filename=package://abilityHand/meshes/idx-F2.STL
- link left_ability_hand_thumb_L1: geometry collision mesh filename=package://abilityHand/meshes/thumb-F1-hull.STL; visual mesh filename=package://abilityHand/meshes/thumb-F1.STL
- link left_ability_hand_thumb_L2: geometry collision mesh filename=package://abilityHand/meshes/thumb-F2-hull.STL; visual mesh filename=package://abilityHand/meshes/thumb-F2-left.STL

File: hand-models/abilityHand/urdf/ability_hand_right_large.urdf (robot description, URDF)
Before this commit: robot right_ability_hand, 46 links, 45 joints
Links:
- link right_ability_hand_base: geometry collision mesh filename=package://abilityHand/meshes/palm_hull_mir.STL; visual mesh filename=package://abilityHand/meshes/FB_palm_ref_MIR.STL
- link right_ability_hand_index_L1: geometry collision mesh filename=package://abilityHand/meshes/idx-F1-hull.STL; visual mesh filename=package://abilityHand/meshes/idx-F1.STL
- link right_ability_hand_index_L2: geometry collision mesh filename=package://abilityHand/meshes/idx-F2-Lg-hull.STL; visual mesh filename=package://abilityHand/meshes/idx-F2-Lg.STL
- link right_ability_hand_middle_L1: geometry collision mesh filename=package://abilityHand/meshes/idx-F1-hull.STL; visual mesh filename=package://abilityHand/meshes/idx-F1.STL
- link right_ability_hand_middle_L2: geometry collision mesh filename=package://abilityHand/meshes/idx-F2-Lg-hull.STL; visual mesh filename=package://abilityHand/meshes/idx-F2-Lg.STL
- link right_ability_hand_pinky_L1: geometry collision mesh filename=package://abilityHand/meshes/idx-F1-hull.STL; visual mesh filename=package://abilityHand/meshes/idx-F1.STL
- link right_ability_hand_pinky_L2: geometry collision mesh filename=package://abilityHand/meshes/idx-F2-hull.STL; visual mesh filename=package://abilityHand/meshes/idx-F2.STL
- link right_ability_hand_ring_L1: geometry collision mesh filename=package://abilityHand/meshes/idx-F1-hull.STL; visual mesh filename=package://abilityHand/meshes/idx-F1.STL
- link right_ability_hand_ring_L2: geometry collision mesh filename=package://abilityHand/meshes/idx-F2-Lg-hull.STL; visual mesh filename=package://abilityHand/meshes/idx-F2-Lg.STL
- link right_ability_hand_thumb_L1: geometry collision mesh filename=package://abilityHand/meshes/thumb-F1-MIR-hull.STL; visual mesh filename=package://abilityHand/meshes/thumb-F1-MIR.STL
- link right_ability_hand_thumb_L2: geometry collision mesh filename=package://abilityHand/meshes/thumb-F2-hull.STL; visual mesh filename=package://abilityHand/meshes/thumb-F2-right.STL
Joints:
- joint right_ability_hand_fsr0: origin xyz=0.02556 -0.01391 -0.00435 rpy=3.14 0 -0.1848 -> xyz=0.02936 -0.01697 -0.00435 rpy=3.14 0 -0.1848
- joint right_ability_hand_fsr1: origin xyz=0.02517 -0.01110 -0.00000 rpy=-1.5708 0.0 -0.2316 -> xyz=0.02961 -0.01394 0.0 rpy=-1.5708 0.0 -0.2316
- joint right_ability_hand_fsr10: origin xyz=0.01310 -0.00943 0.00435 rpy=0.00000 0.00000 -0.57199 -> xyz=0.01472 -0.01099 0.00435 rpy=0.00000 0.00000 -0.57199
- joint right_ability_hand_fsr11: origin xyz=0.03142 -0.01438 0.00000 rpy=-2.66907 -1.57080 0.00000 -> xyz=0.03704 -0.01785 0.00000 rpy=-2.66907 -1.57080 0.00000
- joint right_ability_hand_fsr12: origin xyz=0.02556 -0.01391 -0.00435 rpy=3.14 0 -0.1848 -> xyz=0.02936 -0.01697 -0.00435 rpy=3.14 0 -0.1848
- joint right_ability_hand_fsr13: origin xyz=0.02517 -0.01110 -0.00000 rpy=-1.5708 0.0 -0.2316 -> xyz=0.02961 -0.01394 0.0 rpy=-1.5708 0.0 -0.2316
- joint right_ability_hand_fsr14: origin xyz=0.02556 -0.01391 0.00435 rpy=0.0 0.0 -0.1848036056311012 -> xyz=0.02936 -0.01697 0.00435 rpy=0.0 0.0 -0.1848036056311012
- joint right_ability_hand_fsr15: origin xyz=0.01310 -0.00943 -0.00435 rpy=3.14159 0.00000 -0.57092 -> xyz=0.01472 -0.01100 -0.00435 rpy=3.14159 0.00000 -0.57092
- joint right_ability_hand_fsr16: origin xyz=0.01310 -0.00943 0.00435 rpy=0.00000 0.00000 -0.57199 -> xyz=0.01472 -0.01099 0.00435 rpy=0.00000 0.00000 -0.57199
- joint right_ability_hand_fsr17: origin xyz=0.03142 -0.01438 0.00000 rpy=-2.66907 -1.57080 0.00000 -> xyz=0.03704 -0.01785 0.00000 rpy=-2.66907 -1.57080 0.00000
- joint right_ability_hand_fsr2: origin xyz=0.02556 -0.01391 0.00435 rpy=0.0 0.0 -0.1848036056311012 -> xyz=0.02936 -0.01697 0.00435 rpy=0.0 0.0 -0.1848036056311012
- joint right_ability_hand_fsr3: origin xyz=0.01310 -0.00943 -0.00435 rpy=3.14159 0.00000 -0.57092 -> xyz=0.01472 -0.01100 -0.00435 rpy=3.14159 0.00000 -0.57092
- joint right_ability_hand_fsr4: origin xyz=0.01310 -0.00943 0.00435 rpy=0.00000 0.00000 -0.57199 -> xyz=0.01472 -0.01099 0.00435 rpy=0.00000 0.00000 -0.57199
- joint right_ability_hand_fsr5: origin xyz=0.03142 -0.01438 0.00000 rpy=-2.66907 -1.57080 0.00000 -> xyz=0.03704 -0.01785 0.00000 rpy=-2.66907 -1.57080 0.00000
- joint right_ability_hand_fsr6: origin xyz=0.02556 -0.01391 -0.00435 rpy=3.14 0 -0.1848 -> xyz=0.02936 -0.01697 -0.00435 rpy=3.14 0 -0.1848
- joint right_ability_hand_fsr7: origin xyz=0.02517 -0.01110 -0.00000 rpy=-1.5708 0.0 -0.2316 -> xyz=0.02961 -0.01394 0.0 rpy=-1.5708 0.0 -0.2316
- joint right_ability_hand_fsr8: origin xyz=0.02556 -0.01391 0.00435 rpy=0.0 0.0 -0.1848036056311012 -> xyz=0.02936 -0.01697 0.00435 rpy=0.0 0.0 -0.1848036056311012
- joint right_ability_hand_fsr9: origin xyz=0.01310 -0.00943 -0.00435 rpy=3.14159 0.00000 -0.57092 -> xyz=0.01472 -0.01100 -0.00435 rpy=3.14159 0.00000 -0.57092

File: hand-models/abilityHand/urdf/ability_hand_right_large_no_fsr.urdf (robot description, URDF)
Before this commit: robot right_ability_hand, 46 links, 45 joints
Links:
- removed link right_ability_hand_fsr0
- removed link right_ability_hand_fsr1
- removed link right_ability_hand_fsr10
- removed link right_ability_hand_fsr11
- removed link right_ability_hand_fsr12
- removed link right_ability_hand_fsr13
- removed link right_ability_hand_fsr14
- removed link right_ability_hand_fsr15
- removed link right_ability_hand_fsr16
- removed link right_ability_hand_fsr17
- removed link right_ability_hand_fsr18
- removed link right_ability_hand_fsr19
- removed link right_ability_hand_fsr2
- removed link right_ability_hand_fsr20
- removed link right_ability_hand_fsr21
- removed link right_ability_hand_fsr22
- removed link right_ability_hand_fsr23
- removed link right_ability_hand_fsr24
- removed link right_ability_hand_fsr25
- removed link right_ability_hand_fsr26
- removed link right_ability_hand_fsr27
- removed link right_ability_hand_fsr28
- removed link right_ability_hand_fsr29
- removed link right_ability_hand_fsr3
- removed link right_ability_hand_fsr4
- removed link right_ability_hand_fsr5
- removed link right_ability_hand_fsr6
- removed link right_ability_hand_fsr7
- removed link right_ability_hand_fsr8
- removed link right_ability_hand_fsr9
- link right_ability_hand_base: geometry collision mesh filename=package://abilityHand/meshes/palm_hull_mir.STL; visual mesh filename=package://abilityHand/meshes/FB_palm_ref_MIR.STL
- link right_ability_hand_index_L1: geometry collision mesh filename=package://abilityHand/meshes/idx-F1-hull.STL; visual mesh filename=package://abilityHand/meshes/idx-F1.STL
- link right_ability_hand_index_L2: geometry collision mesh filename=package://abilityHand/meshes/idx-F2-Lg-hull.STL; visual mesh filename=package://abilityHand/meshes/idx-F2-Lg.STL
- link right_ability_hand_middle_L1: geometry collision mesh filename=package://abilityHand/meshes/idx-F1-hull.STL; visual mesh filename=package://abilityHand/meshes/idx-F1.STL
- link right_ability_hand_middle_L2: geometry collision mesh filename=package://abilityHand/meshes/idx-F2-Lg-hull.STL; visual mesh filename=package://abilityHand/meshes/idx-F2-Lg.STL
- link right_ability_hand_pinky_L1: geometry collision mesh filename=package://abilityHand/meshes/idx-F1-hull.STL; visual mesh filename=package://abilityHand/meshes/idx-F1.STL
- link right_ability_hand_pinky_L2: geometry collision mesh filename=package://abilityHand/meshes/idx-F2-hull.STL; visual mesh filename=package://abilityHand/meshes/idx-F2.STL
- link right_ability_hand_ring_L1: geometry collision mesh filename=package://abilityHand/meshes/idx-F1-hull.STL; visual mesh filename=package://abilityHand/meshes/idx-F1.STL
- link right_ability_hand_ring_L2: geometry collision mesh filename=package://abilityHand/meshes/idx-F2-Lg-hull.STL; visual mesh filename=package://abilityHand/meshes/idx-F2-Lg.STL
- link right_ability_hand_thumb_L1: geometry collision mesh filename=package://abilityHand/meshes/thumb-F1-MIR-hull.STL; visual mesh filename=package://abilityHand/meshes/thumb-F1-MIR.STL
- link right_ability_hand_thumb_L2: geometry collision mesh filename=package://abilityHand/meshes/thumb-F2-hull.STL; visual mesh filename=package://abilityHand/meshes/thumb-F2-right.STL
Joints:
- removed joint right_ability_hand_fsr0
- removed joint right_ability_hand_fsr1
- removed joint right_ability_hand_fsr10
- removed joint right_ability_hand_fsr11
- removed joint right_ability_hand_fsr12
- removed joint right_ability_hand_fsr13
- removed joint right_ability_hand_fsr14
- removed joint right_ability_hand_fsr15
- removed joint right_ability_hand_fsr16
- removed joint right_ability_hand_fsr17
- removed joint right_ability_hand_fsr18
- removed joint right_ability_hand_fsr19
- removed joint right_ability_hand_fsr2
- removed joint right_ability_hand_fsr20
- removed joint right_ability_hand_fsr21
- removed joint right_ability_hand_fsr22
- removed joint right_ability_hand_fsr23
- removed joint right_ability_hand_fsr24
- removed joint right_ability_hand_fsr25
- removed joint right_ability_hand_fsr26
- removed joint right_ability_hand_fsr27
- removed joint right_ability_hand_fsr28
- removed joint right_ability_hand_fsr29
- removed joint right_ability_hand_fsr3
- removed joint right_ability_hand_fsr4
- removed joint right_ability_hand_fsr5
- removed joint right_ability_hand_fsr6
- removed joint right_ability_hand_fsr7
- removed joint right_ability_hand_fsr8
- removed joint right_ability_hand_fsr9

File: hand-models/abilityHand/urdf/ability_hand_right_small.urdf (robot description, URDF)
Before this commit: robot right_ability_hand, 16 links, 15 joints
Links:
- added link right_ability_hand_fsr0
- added link right_ability_hand_fsr1
- added link right_ability_hand_fsr10
- added link right_ability_hand_fsr11
- added link right_ability_hand_fsr12
- added link right_ability_hand_fsr13
- added link right_ability_hand_fsr14
- added link right_ability_hand_fsr15
- added link right_ability_hand_fsr16
- added link right_ability_hand_fsr17
- added link right_ability_hand_fsr18
- added link right_ability_hand_fsr19
- added link right_ability_hand_fsr2
- added link right_ability_hand_fsr20
- added link right_ability_hand_fsr21
- added link right_ability_hand_fsr22
- added link right_ability_hand_fsr23
- added link right_ability_hand_fsr24
- added link right_ability_hand_fsr25
- added link right_ability_hand_fsr26
- added link right_ability_hand_fsr27
- added link right_ability_hand_fsr28
- added link right_ability_hand_fsr29
- added link right_ability_hand_fsr3
- added link right_ability_hand_fsr4
- added link right_ability_hand_fsr5
- added link right_ability_hand_fsr6
- added link right_ability_hand_fsr7
- added link right_ability_hand_fsr8
- added link right_ability_hand_fsr9
- link right_ability_hand_base: geometry collision mesh filename=package://abilityHand/meshes/palm_hull_mir.STL; visual mesh filename=package://abilityHand/meshes/FB_palm_ref_MIR.STL
- link right_ability_hand_index_L1: geometry collision mesh filename=package://abilityHand/meshes/idx-F1-hull.STL; visual mesh filename=package://abilityHand/meshes/idx-F1.STL
- link right_ability_hand_index_L2: geometry collision mesh filename=package://abilityHand/meshes/idx-F2-hull.STL; visual mesh filename=package://abilityHand/meshes/idx-F2.STL
- link right_ability_hand_middle_L1: geometry collision mesh filename=package://abilityHand/meshes/idx-F1-hull.STL; visual mesh filename=package://abilityHand/meshes/idx-F1.STL
- link right_ability_hand_middle_L2: geometry collision mesh filename=package://abilityHand/meshes/idx-F2-hull.STL; visual mesh filename=package://abilityHand/meshes/idx-F2.STL
- link right_ability_hand_pinky_L1: geometry collision mesh filename=package://abilityHand/meshes/idx-F1-hull.STL; visual mesh filename=package://abilityHand/meshes/idx-F1.STL
- link right_ability_hand_pinky_L2: geometry collision mesh filename=package://abilityHand/meshes/idx-F2-hull.STL; visual mesh filename=package://abilityHand/meshes/idx-F2.STL
- link right_ability_hand_ring_L1: geometry collision mesh filename=package://abilityHand/meshes/idx-F1-hull.STL; visual mesh filename=package://abilityHand/meshes/idx-F1.STL
- link right_ability_hand_ring_L2: geometry collision mesh filename=package://abilityHand/meshes/idx-F2-hull.STL; visual mesh filename=package://abilityHand/meshes/idx-F2.STL
- link right_ability_hand_thumb_L1: geometry collision mesh filename=package://abilityHand/meshes/thumb-F1-MIR-hull.STL; visual mesh filename=package://abilityHand/meshes/thumb-F1-MIR.STL
- link right_ability_hand_thumb_L2: geometry collision mesh filename=package://abilityHand/meshes/thumb-F2-hull.STL; visual mesh filename=package://abilityHand/meshes/thumb-F2-right.STL
Joints:
- added joint right_ability_hand_fsr0: type fixed, parent right_ability_hand_index_L2, child right_ability_hand_fsr0, origin xyz=0.02556 -0.01391 -0.00435 rpy=3.14 0 -0.1848
- added joint right_ability_hand_fsr1: type fixed, parent right_ability_hand_index_L2, child right_ability_hand_fsr1, origin xyz=0.02517 -0.01110 -0.00000 rpy=-1.5708 0.0 -0.2316
- added joint right_ability_hand_fsr10: type fixed, parent right_ability_hand_middle_L2, child right_ability_hand_fsr10, origin xyz=0.01310 -0.00943 0.00435 rpy=0.00000 0.00000 -0.57199
- added joint right_ability_hand_fsr11: type fixed, parent right_ability_hand_middle_L2, child right_ability_hand_fsr11, origin xyz=0.03142 -0.01438 0.00000 rpy=-2.66907 -1.57080 0.00000
- added joint right_ability_hand_fsr12: type fixed, parent right_ability_hand_ring_L2, child right_ability_hand_fsr12, origin xyz=0.02556 -0.01391 -0.00435 rpy=3.14 0 -0.1848
- added joint right_ability_hand_fsr13: type fixed, parent right_ability_hand_ring_L2, child right_ability_hand_fsr13, origin xyz=0.02517 -0.01110 -0.00000 rpy=-1.5708 0.0 -0.2316
- added joint right_ability_hand_fsr14: type fixed, parent right_ability_hand_ring_L2, child right_ability_hand_fsr14, origin xyz=0.02556 -0.01391 0.00435 rpy=0.0 0.0 -0.1848036056311012
- added joint right_ability_hand_fsr15: type fixed, parent right_ability_hand_ring_L2, child right_ability_hand_fsr15, origin xyz=0.01310 -0.00943 -0.00435 rpy=3.14159 0.00000 -0.57092
- added joint right_ability_hand_fsr16: type fixed, parent right_ability_hand_ring_L2, child right_ability_hand_fsr16, origin xyz=0.01310 -0.00943 0.00435 rpy=0.00000 0.00000 -0.57199
- added joint right_ability_hand_fsr17: type fixed, parent right_ability_hand_ring_L2, child right_ability_hand_fsr17, origin xyz=0.03142 -0.01438 0.00000 rpy=-2.66907 -1.57080 0.00000
- added joint right_ability_hand_fsr18: type fixed, parent right_ability_hand_pinky_L2, child right_ability_hand_fsr18, origin xyz=0.02556 -0.01391 -0.00435 rpy=3.14 0 -0.1848
- added joint right_ability_hand_fsr19: type fixed, parent right_ability_hand_pinky_L2, child right_ability_hand_fsr19, origin xyz=0.02517 -0.01110 -0.00000 rpy=-1.5708 0.0 -0.2316
- added joint right_ability_hand_fsr2: type fixed, parent right_ability_hand_index_L2, child right_ability_hand_fsr2, origin xyz=0.02556 -0.01391 0.00435 rpy=0.0 0.0 -0.1848036056311012
- added joint right_ability_hand_fsr20: type fixed, parent right_ability_hand_pinky_L2, child right_ability_hand_fsr20, origin xyz=0.02556 -0.01391 0.00435 rpy=0.0 0.0 -0.1848036056311012
- added joint right_ability_hand_fsr21: type fixed, parent right_ability_hand_pinky_L2, child right_ability_hand_fsr21, origin xyz=0.01310 -0.00943 -0.00435 rpy=3.14159 0.00000 -0.57092
- added joint right_ability_hand_fsr22: type fixed, parent right_ability_hand_pinky_L2, child right_ability_hand_fsr22, origin xyz=0.01310 -0.00943 0.00435 rpy=0.00000 0.00000 -0.57199
- added joint right_ability_hand_fsr23: type fixed, parent right_ability_hand_pinky_L2, child right_ability_hand_fsr23, origin xyz=0.03142 -0.01438 0.00000 rpy=-2.66907 -1.57080 0.00000
- added joint right_ability_hand_fsr24: type fixed, parent right_ability_hand_thumb_L2, child right_ability_hand_fsr24, origin xyz=0.04747 0.01988 -0.001239 rpy=-2.29074 0.00001 0.41769
- added joint right_ability_hand_fsr25: type fixed, parent right_ability_hand_thumb_L2, child right_ability_hand_fsr25, origin xyz=0.04721 0.02124 0.006439 rpy=-1.30899 0.00001 0.41769
- added joint right_ability_hand_fsr26: type fixed, parent right_ability_hand_thumb_L2, child right_ability_hand_fsr26, origin xyz=0.04896 0.01654 0.01241 rpy=-0.32726 0.00001 0.41769
- added joint right_ability_hand_fsr27: type fixed, parent right_ability_hand_thumb_L2, child right_ability_hand_fsr27, origin xyz=0.03739 0.01536 -0.001289 rpy=-2.29074 0.00001 0.41769
- added joint right_ability_hand_fsr28: type fixed, parent right_ability_hand_thumb_L2, child right_ability_hand_fsr28, origin xyz=0.03888 0.01200 0.01244 rpy=-0.32726 0.00001 0.41769
- added joint right_ability_hand_fsr29: type fixed, parent right_ability_hand_thumb_L2, child right_ability_hand_fsr29, origin xyz=0.05591 0.02160 0.00558
- added joint right_ability_hand_fsr3: type fixed, parent right_ability_hand_index_L2, child right_ability_hand_fsr3, origin xyz=0.01310 -0.00943 -0.00435 rpy=3.14159 0.00000 -0.57092
- added joint right_ability_hand_fsr4: type fixed, parent right_ability_hand_index_L2, child right_ability_hand_fsr4, origin xyz=0.01310 -0.00943 0.00435 rpy=0.00000 0.00000 -0.57199
- added joint right_ability_hand_fsr5: type fixed, parent right_ability_hand_index_L2, child right_ability_hand_fsr5, origin xyz=0.03142 -0.01438 0.00000 rpy=-2.66907 -1.57080 0.00000
- added joint right_ability_hand_fsr6: type fixed, parent right_ability_hand_middle_L2, child right_ability_hand_fsr6, origin xyz=0.02556 -0.01391 -0.00435 rpy=3.14 0 -0.1848
- added joint right_ability_hand_fsr7: type fixed, parent right_ability_hand_middle_L2, child right_ability_hand_fsr7, origin xyz=0.02517 -0.01110 -0.00000 rpy=-1.5708 0.0 -0.2316
- added joint right_ability_hand_fsr8: type fixed, parent right_ability_hand_middle_L2, child right_ability_hand_fsr8, origin xyz=0.02556 -0.01391 0.00435 rpy=0.0 0.0 -0.1848036056311012
- added joint right_ability_hand_fsr9: type fixed, parent right_ability_hand_middle_L2, child right_ability_hand_fsr9, origin xyz=0.01310 -0.00943 -0.00435 rpy=3.14159 0.00000 -0.57092
