Commit message: modified hand urdf/mesh paths to be consistant with our typical system

File: hand-models/ezGripper/urdf/left_ezgripper_gen2.urdf (robot description, URDF)
Before this commit: robot right_ezgripper_gen2, 5 links, 4 joints
Links:
- removed link right_ezgripper_finger_l1_1
- removed link right_ezgripper_finger_l1_2
- removed link right_ezgripper_finger_l2_1
- removed link right_ezgripper_finger_l2_2
- removed link right_ezgripper_palm_link
- added link left_ezgripper_finger_l1_1, mass 0.025; collision mesh filename=package://ezGripper/meshes/ezgripper_gen2/SAKE_Finger_L1_Ge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; visual mesh filename=package://ezGripper/meshes/ezgripper_gen2/SAKE_Finger_L1_Ge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
- added link left_ezgripper_finger_l1_2, mass 0.025; collision mesh filename=package://ezGripper/meshes/ezgripper_gen2/SAKE_Finger_L1_Ge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; visual mesh filename=package://ezGripper/meshes/ezgripper_gen2/SAKE_Finger_L1_Ge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
- added link left_ezgripper_finger_l2_1, mass .025; collision mesh filename=package://ezGripper/meshes/ezgripper_gen2/SAKE_Finger_L2_Ge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; visual mesh filename=package://ezGripper/meshes/ezgripper_gen2/SAKE_Finger_L2_Ge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
- added link left_ezgripper_finger_l2_2, mass .025; collision mesh filename=package://ezGripper/meshes/ezgripper_gen2/SAKE_Finger_L2_Ge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; visual mesh filename=package://ezGripper/meshes/ezgripper_gen2/SAKE_Finger_L2_Ge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
- added link left_ezgripper_palm_link, mass 0.3; collision mesh filename=package://ezGripper/meshes/ezgripper_gen2/SAKE_Palm_Dual_Ge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; visual mesh filename=package://ezGripper/meshes/ezgripper_gen2/SAKE_Palm_Dual_Ge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
Joints:
- removed joint right_ezgripper_knuckle_l1_l2_1
- removed joint right_ezgripper_knuckle_l1_l2_2
- removed joint right_ezgripper_knuckle_palm_l1_1
- removed joint right_ezgripper_knuckle_palm_l1_2
- added joint left_ezgripper_knuckle_l1_l2_1: type revolute, parent left_ezgripper_finger_l1_1, child left_ezgripper_finger_l2_1, origin xyz=0.052 0 0 rpy=0 0 0, axis 0 1 0, limit lower=0 upper=1.94 effort=1 velocity=3.67
- added joint left_ezgripper_knuckle_l1_l2_2: type revolute, parent left_ezgripper_finger_l1_2, child left_ezgripper_finger_l2_2, origin xyz=0.052 0 0 rpy=0 0 0, axis 0 1 0, limit lower=0 upper=1.94 effort=1 velocity=3.67, mimic joint=left_ezgripper_knuckle_l1_l2_1
- added joint left_ezgripper_knuckle_palm_l1_1: type revolute, parent left_ezgripper_palm_link, child left_ezgripper_finger_l1_1, origin xyz=0.072569 0.03 0 rpy=-1.5708 0 1.57075, axis 0 1 0, limit lower=0 upper=1.94 effort=1 velocity=3.67
- added joint left_ezgripper_knuckle_palm_l1_2: type revolute, parent left_ezgripper_palm_link, child left_ezgripper_finger_l1_2, origin xyz=0.072569 -0.03 0 rpy=1.5708 0 -1.57075, axis 0 1 0, limit lower=0 upper=1.94 effort=1 velocity=3.67, mimic joint=left_ezgripper_knuckle_palm_l1_1

File: hand-models/ezGripper/urdf/right_ezgripper_gen2.urdf (robot description, URDF)
Before this commit: robot left_ezgripper_gen2, 5 links, 4 joints
Links:
- removed link left_ezgripper_finger_l1_1
- removed link left_ezgripper_finger_l1_2
- removed link left_ezgripper_finger_l2_1
- removed link left_ezgripper_finger_l2_2
- removed link left_ezgripper_palm_link
- added link right_ezgripper_finger_l1_1, mass 0.025; collision mesh filename=package://ezGripper/meshes/ezgripper_gen2/SAKE_Finger_L1_Ge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; visual mesh filename=package://ezGripper/meshes/ezgripper_gen2/SAKE_Finger_L1_Ge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
- added link right_ezgripper_finger_l1_2, mass 0.025; collision mesh filename=package://ezGripper/meshes/ezgripper_gen2/SAKE_Finger_L1_Ge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; visual mesh filename=package://ezGripper/meshes/ezgripper_gen2/SAKE_Finger_L1_Ge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
- added link right_ezgripper_finger_l2_1, mass .025; collision mesh filename=package://ezGripper/meshes/ezgripper_gen2/SAKE_Finger_L2_Ge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; visual mesh filename=package://ezGripper/meshes/ezgripper_gen2/SAKE_Finger_L2_Ge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
- added link right_ezgripper_finger_l2_2, mass .025; collision mesh filename=package://ezGripper/meshes/ezgripper_gen2/SAKE_Finger_L2_Ge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; visual mesh filename=package://ezGripper/meshes/ezgripper_gen2/SAKE_Finger_L2_Ge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
- added link right_ezgripper_palm_link, mass 0.3; collision mesh filename=package://ezGripper/meshes/ezgripper_gen2/SAKE_Palm_Dual_Ge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; visual mesh filename=package://ezGripper/meshes/ezgripper_gen2/SAKE_Palm_Dual_Ge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
Joints:
- removed joint left_ezgripper_knuckle_l1_l2_1
- removed joint left_ezgripper_knuckle_l1_l2_2
- removed joint left_ezgripper_knuckle_palm_l1_1
- removed joint left_ezgripper_knuckle_palm_l1_2
- added joint right_ezgripper_knuckle_l1_l2_1: type revolute, parent right_ezgripper_finger_l1_1, child right_ezgripper_finger_l2_1, origin xyz=0.052 0 0 rpy=0 0 0, axis 0 1 0, limit lower=0 upper=1.94 effort=1 velocity=3.67
- added joint right_ezgripper_knuckle_l1_l2_2: type revolute, parent right_ezgripper_finger_l1_2, child right_ezgripper_finger_l2_2, origin xyz=0.052 0 0 rpy=0 0 0, axis 0 1 0, limit lower=0 upper=1.94 effort=1 velocity=3.67, mimic joint=right_ezgripper_knuckle_l1_l2_1
- added joint right_ezgripper_knuckle_palm_l1_1: type revolute, parent right_ezgripper_palm_link, child right_ezgripper_finger_l1_1, origin xyz=0.072569 0.03 0 rpy=-1.5708 0 1.57075, axis 0 1 0, limit lower=0 upper=1.94 effort=1 velocity=3.67
- added joint right_ezgripper_knuckle_palm_l1_2: type revolute, parent right_ezgripper_palm_link, child right_ezgripper_finger_l1_2, origin xyz=0.072569 -0.03 0 rpy=1.5708 0 -1.57075, axis 0 1 0, limit lower=0 upper=1.94 effort=1 velocity=3.67, mimic joint=right_ezgripper_knuckle_palm_l1_1

Commit message: Converted STL files to OBJs

File: hand-models/abilityHand/urdf/ability_hand_left_large.urdf (robot description, URDF)
Before this commit: robot left_ability_hand, 46 links, 45 joints
Links:
- link left_ability_hand_base: geometry collision mesh filename=package://abilityHand/meshes/palm_hull.obj; visual mesh filename=package://abilityHand/meshes/FB_palm_ref.obj
- link left_ability_hand_index_L1: geometry collision mesh filename=package://abilityHand/meshes/idx-F1-hull.obj; visual mesh filename=package://abilityHand/meshes/idx-F1.obj
- link left_ability_hand_index_L2: geometry collision mesh filename=package://abilityHand/meshes/idx-F2-Lg-hull.obj; visual mesh filename=package://abilityHand/meshes/idx-F2-Lg.obj
- link left_ability_hand_middle_L1: geometry collision mesh filename=package://abilityHand/meshes/idx-F1-hull.obj; visual mesh filename=package://abilityHand/meshes/idx-F1.obj
- link left_ability_hand_middle_L2: geometry collision mesh filename=package://abilityHand/meshes/idx-F2-Lg-hull.obj; visual mesh filename=package://abilityHand/meshes/idx-F2-Lg.obj
- link left_ability_hand_pinky_L1: geometry collision mesh filename=package://abilityHand/meshes/idx-F1-hull.obj; visual mesh filename=package://abilityHand/meshes/idx-F1.obj
- link left_ability_hand_pinky_L2: geometry collision mesh filename=package://abilityHand/meshes/idx-F2-hull.obj; visual mesh filename=package://abilityHand/meshes/idx-F2-Lg.obj
- link left_ability_hand_ring_L1: geometry collision mesh filename=package://abilityHand/meshes/idx-F1-hull.obj; visual mesh filename=package://abilityHand/meshes/idx-F1.obj
- link left_ability_hand_ring_L2: geometry collision mesh filename=package://abilityHand/meshes/idx-F2-Lg-hull.obj; visual mesh filename=package://abilityHand/meshes/idx-F2-Lg.obj
- link left_ability_hand_thumb_L1: geometry collision mesh filename=package://abilityHand/meshes/thumb-F1-hull.obj; visual mesh filename=package://abilityHand/meshes/thumb-F1.obj
- link left_ability_hand_thumb_L2: geometry collision mesh filename=package://abilityHand/meshes/thumb-F2-hull.obj; visual mesh filename=package://abilityHand/meshes/thumb-F2-left.obj

File: hand-models/abilityHand/urdf/ability_hand_left_small.urdf (robot description, URDF)
Before this commit: robot left_ability_hand, 46 links, 45 joints
Links:
- link left_ability_hand_base: geometry collision mesh filename=package://abilityHand/meshes/palm_hull.obj; visual mesh filename=package://abilityHand/meshes/FB_palm_ref.obj
- link left_ability_hand_index_L1: geometry collision mesh filename=package://abilityHand/meshes/idx-F1-hull.obj; visual mesh filename=package://abilityHand/meshes/idx-F1.obj
- link left_ability_hand_index_L2: geometry collision mesh filename=package://abilityHand/meshes/idx-F2-hull.obj; visual mesh filename=package://abilityHand/meshes/idx-F2.obj
- link left_ability_hand_middle_L1: geometry collision mesh filename=package://abilityHand/meshes/idx-F1-hull.obj; visual mesh filename=package://abilityHand/meshes/idx-F1.obj
- link left_ability_hand_middle_L2: geometry collision mesh filename=package://abilityHand/meshes/idx-F2-hull.obj; visual mesh filename=package://abilityHand/meshes/idx-F2.obj
- link left_ability_hand_pinky_L1: geometry collision mesh filename=package://abilityHand/meshes/idx-F1-hull.obj; visual mesh filename=package://abilityHand/meshes/idx-F1.obj
- link left_ability_hand_pinky_L2: geometry collision mesh filename=package://abilityHand/meshes/idx-F2-hull.obj; visual mesh filename=package://abilityHand/meshes/idx-F2.obj
- link left_ability_hand_ring_L1: geometry collision mesh filename=package://abilityHand/meshes/idx-F1-hull.obj; visual mesh filename=package://abilityHand/meshes/idx-F1.obj
- link left_ability_hand_ring_L2: geometry collision mesh filename=package://abilityHand/meshes/idx-F2-hull.obj; visual mesh filename=package://abilityHand/meshes/idx-F2.obj
- link left_ability_hand_thumb_L1: geometry collision mesh filename=package://abilityHand/meshes/thumb-F1-hull.obj; visual mesh filename=package://abilityHand/meshes/thumb-F1.obj
- link left_ability_hand_thumb_L2: geometry collision mesh filename=package://abilityHand/meshes/thumb-F2-hull.obj; visual mesh filename=package://abilityHand/meshes/thumb-F2-left.obj

File: hand-models/abilityHand/urdf/ability_hand_right_large.urdf (robot description, URDF)
Before this commit: robot right_ability_hand, 46 links, 45 joints
Links:
- link right_ability_hand_base: geometry collision mesh filename=package://abilityHand/meshes/palm_hull_mir.obj; visual mesh filename=package://abilityHand/meshes/FB_palm_ref_MIR.obj
- link right_ability_hand_index_L1: geometry collision mesh filename=package://abilityHand/meshes/idx-F1-hull.obj; visual mesh filename=package://abilityHand/meshes/idx-F1.obj
- link right_ability_hand_index_L2: geometry collision mesh filename=package://abilityHand/meshes/idx-F2-Lg-hull.obj; visual mesh filename=package://abilityHand/meshes/idx-F2-Lg.obj
- link right_ability_hand_middle_L1: geometry collision mesh filename=package://abilityHand/meshes/idx-F1-hull.obj; visual mesh filename=package://abilityHand/meshes/idx-F1.obj
- link right_ability_hand_middle_L2: geometry collision mesh filename=package://abilityHand/meshes/idx-F2-Lg-hull.obj; visual mesh filename=package://abilityHand/meshes/idx-F2-Lg.obj
- link right_ability_hand_pinky_L1: geometry collision mesh filename=package://abilityHand/meshes/idx-F1-hull.obj; visual mesh filename=package://abilityHand/meshes/idx-F1.obj
- link right_ability_hand_pinky_L2: geometry collision mesh filename=package://abilityHand/meshes/idx-F2-hull.obj; visual mesh filename=package://abilityHand/meshes/idx-F2.obj
- link right_ability_hand_ring_L1: geometry collision mesh filename=package://abilityHand/meshes/idx-F1-hull.obj; visual mesh filename=package://abilityHand/meshes/idx-F1.obj
- link right_ability_hand_ring_L2: geometry collision mesh filename=package://abilityHand/meshes/idx-F2-Lg-hull.obj; visual mesh filename=package://abilityHand/meshes/idx-F2-Lg.obj
- link right_ability_hand_thumb_L1: geometry collision mesh filename=package://abilityHand/meshes/thumb-F1-MIR-hull.obj; visual mesh filename=package://abilityHand/meshes/thumb-F1-MIR.obj
- link right_ability_hand_thumb_L2: geometry collision mesh filename=package://abilityHand/meshes/thumb-F2-hull.obj; visual mesh filename=package://abilityHand/meshes/thumb-F2-right.obj

File: hand-models/abilityHand/urdf/ability_hand_right_large_no_fsr.urdf (robot description, URDF)
Before this commit: robot right_ability_hand, 16 links, 15 joints
Links:
- link right_ability_hand_base: geometry collision mesh filename=package://abilityHand/meshes/palm_hull_mir.obj; visual mesh filename=package://abilityHand/meshes/FB_palm_ref_MIR.obj
- link right_ability_hand_index_L1: geometry collision mesh filename=package://abilityHand/meshes/idx-F1-hull.obj; visual mesh filename=package://abilityHand/meshes/idx-F1.obj
- link right_ability_hand_index_L2: geometry collision mesh filename=package://abilityHand/meshes/idx-F2-Lg-hull.obj; visual mesh filename=package://abilityHand/meshes/idx-F2-Lg.obj
- link right_ability_hand_middle_L1: geometry collision mesh filename=package://abilityHand/meshes/idx-F1-hull.obj; visual mesh filename=package://abilityHand/meshes/idx-F1.obj
- link right_ability_hand_middle_L2: geometry collision mesh filename=package://abilityHand/meshes/idx-F2-Lg-hull.obj; visual mesh filename=package://abilityHand/meshes/idx-F2-Lg.obj
- link right_ability_hand_pinky_L1: geometry collision mesh filename=package://abilityHand/meshes/idx-F1-hull.obj; visual mesh filename=package://abilityHand/meshes/idx-F1.obj
- link right_ability_hand_pinky_L2: geometry collision mesh filename=package://abilityHand/meshes/idx-F2-hull.obj; visual mesh filename=package://abilityHand/meshes/idx-F2.obj
- link right_ability_hand_ring_L1: geometry collision mesh filename=package://abilityHand/meshes/idx-F1-hull.obj; visual mesh filename=package://abilityHand/meshes/idx-F1.obj
- link right_ability_hand_ring_L2: geometry collision mesh filename=package://abilityHand/meshes/idx-F2-Lg-hull.obj; visual mesh filename=package://abilityHand/meshes/idx-F2-Lg.obj
- link right_ability_hand_thumb_L1: geometry collision mesh filename=package://abilityHand/meshes/thumb-F1-MIR-hull.obj; visual mesh filename=package://abilityHand/meshes/thumb-F1-MIR.obj
- link right_ability_hand_thumb_L2: geometry collision mesh filename=package://abilityHand/meshes/thumb-F2-hull.obj; visual mesh filename=package://abilityHand/meshes/thumb-F2-right.obj

File: hand-models/abilityHand/urdf/ability_hand_right_small.urdf (robot description, URDF)
Before this commit: robot right_ability_hand, 46 links, 45 joints
Links:
- link right_ability_hand_base: geometry collision mesh filename=package://abilityHand/meshes/palm_hull_mir.obj; visual mesh filename=package://abilityHand/meshes/FB_palm_ref_MIR.obj
- link right_ability_hand_index_L1: geometry collision mesh filename=package://abilityHand/meshes/idx-F1-hull.obj; visual mesh filename=package://abilityHand/meshes/idx-F1.obj
- link right_ability_hand_index_L2: geometry collision mesh filename=package://abilityHand/meshes/idx-F2-hull.obj; visual mesh filename=package://abilityHand/meshes/idx-F2.obj
- link right_ability_hand_middle_L1: geometry collision mesh filename=package://abilityHand/meshes/idx-F1-hull.obj; visual mesh filename=package://abilityHand/meshes/idx-F1.obj
- link right_ability_hand_middle_L2: geometry collision mesh filename=package://abilityHand/meshes/idx-F2-hull.obj; visual mesh filename=package://abilityHand/meshes/idx-F2.obj
- link right_ability_hand_pinky_L1: geometry collision mesh filename=package://abilityHand/meshes/idx-F1-hull.obj; visual mesh filename=package://abilityHand/meshes/idx-F1.obj
- link right_ability_hand_pinky_L2: geometry collision mesh filename=package://abilityHand/meshes/idx-F2-hull.obj; visual mesh filename=package://abilityHand/meshes/idx-F2.obj
- link right_ability_hand_ring_L1: geometry collision mesh filename=package://abilityHand/meshes/idx-F1-hull.obj; visual mesh filename=package://abilityHand/meshes/idx-F1.obj
- link right_ability_hand_ring_L2: geometry collision mesh filename=package://abilityHand/meshes/idx-F2-hull.obj; visual mesh filename=package://abilityHand/meshes/idx-F2.obj
- link right_ability_hand_thumb_L1: geometry collision mesh filename=package://abilityHand/meshes/thumb-F1-MIR-hull.obj; visual mesh filename=package://abilityHand/meshes/thumb-F1-MIR.obj
- link right_ability_hand_thumb_L2: geometry collision mesh filename=package://abilityHand/meshes/thumb-F2-hull.obj; visual mesh filename=package://abilityHand/meshes/thumb-F2-right.obj
